Commit message: gazebo pkg

File: src/tamrin_robot/description/robot_core.xacro (robot description, xacro)
@@ -48,4 +48,7 @@
         </xacro:inertial_box>
     </link>
+    <gazebo reference="shaft_link">
+        <material>Gazebo/Blue</material>
+    </gazebo>
     <joint name="base_shaft_joint" type="fixed">
         <origin xyz="0 0 ${L1 + LW/2}" rpy="0 0 0"/>
@@ -72,4 +75,7 @@
         </xacro:inertial_box>
     </link>
+    <gazebo reference="left_leg_link">
+        <material>Gazebo/Orange</material>
+    </gazebo>
     <joint name="left_leg_joint" type="fixed">
         <origin xyz="0 ${W/2} ${-L1}" rpy="0 0 0"/>
@@ -96,4 +102,7 @@
         </xacro:inertial_cylinder>
     </link>
+    <gazebo reference="left_wheel_link">
+        <material>Gazebo/White</material>
+    </gazebo>
     <joint name="left_wheel_joint" type="${motor}">
         <origin xyz="0 ${LW/2 + WL/2 + 0.002} 0" rpy="${-pi/2} 0 0"/>
@@ -121,4 +130,7 @@
         </xacro:inertial_box>
     </link>
+    <gazebo reference="right_leg_link">
+        <material>Gazebo/Orange</material>
+    </gazebo>
     <joint name="right_leg_joint" type="fixed">
         <origin xyz="0 ${-W/2} ${-L1}" rpy="0 0 0"/>
@@ -145,4 +157,7 @@
         </xacro:inertial_cylinder>
     </link>
+    <gazebo reference="right_wheel_link">
+        <material>Gazebo/White</material>
+    </gazebo>
     <joint name="right_wheel_joint" type="${motor}">
         <origin xyz="0 ${-LW/2 - WL/2 - 0.002} 0" rpy="${pi/2} 0 0"/>
@@ -170,4 +185,7 @@
         </xacro:inertial_box>
     </link>
+    <gazebo reference="left_hand_link">
+        <material>Gazebo/Orange</material>
+    </gazebo>
     <joint name="left_hand_joint" type="fixed">
         <origin xyz="0 ${W/2 + LW} 0" rpy="0 ${-pi/2} 0"/>
@@ -194,4 +212,7 @@
         </xacro:inertial_box>
     </link>
+    <gazebo reference="right_hand_link">
+        <material>Gazebo/Orange</material>
+    </gazebo>
     <joint name="right_hand_joint" type="fixed">
         <origin xyz="0 ${-W/2 - LW} 0" rpy="0 ${-pi/2} 0"/>
